Commit message: testing

File: assets/urdf/franka_description/franka_panda_no_gripper.urdf (robot description, URDF)
Before this commit: robot panda, 13 links, 12 joints
Links:
- link panda_link2: geometry collision mesh filename=package://franka_motion_control/assets/urdf/franka_descript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; visual mesh filename=$(find franka_motion_control)assets/urdf/franka_description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

Commit message: changes to urdf

File: assets/urdf/franka_description/franka_panda_no_gripper.urdf (robot description, URDF)
Before this commit: robot panda, 13 links, 12 joints
Links:
- link panda_link2: geometry collision mesh filename=$(find franka_motion_control)/assets/urdf/franka_descriptio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; visual mesh filename=$(find franka_motion_control)/assets/urdf/franka_descriptio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

Commit message: changes to urdf

File: assets/urdf/franka_description/franka_panda_no_gripper.urdf (robot description, URDF)
Before this commit: robot panda, 13 links, 12 joints
Links:
- link panda_link0: geometry collision mesh filename=$(find franka_motion_control)/assets/urdf/franka_descriptio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; visual mesh filename=$(find franka_motion_control)/assets/urdf/franka_descriptio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
- link panda_link1: geometry collision mesh filename=$(find franka_motion_control)/assets/urdf/franka_descriptio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; visual mesh filename=$(find franka_motion_control)/assets/urdf/franka_descriptio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
- link panda_link3: geometry collision mesh filename=$(find franka_motion_control)/assets/urdf/franka_descriptio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; visual mesh filename=$(find franka_motion_control)/assets/urdf/franka_descriptio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

Commit message: more changes to urdf

File: assets/urdf/franka_description/franka_panda_no_gripper.urdf (robot description, URDF)
Before this commit: robot panda, 13 links, 12 joints
Links:
- link panda_hand: geometry collision mesh filename=package://franka_motion_control/assets/urdf/franka_descript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; visual mesh filename=package://franka_motion_control/assets/urdf/franka_descript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
- link panda_leftfinger: geometry collision mesh filename=package://franka_motion_control/assets/urdf/franka_descript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; visual mesh filename=package://franka_motion_control/assets/urdf/franka_descript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
- link panda_link0: geometry collision mesh filename=package://franka_motion_control/assets/urdf/franka_descript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; visual mesh filename=package://franka_motion_control/assets/urdf/franka_descript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
- link panda_link1: geometry collision mesh filename=package://franka_motion_control/assets/urdf/franka_descript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; visual mesh filename=package://franka_motion_control/assets/urdf/franka_descript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
- link panda_link2: geometry collision mesh filename=$package://franka_motion_control/assets/urdf/franka_descrip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; visual mesh filename=$package://franka_motion_control/assets/urdf/franka_descrip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
- link panda_link3: geometry collision mesh filename=package://franka_motion_control/assets/urdf/franka_descript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; visual mesh filename=package://franka_motion_control/assets/urdf/franka_descript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
- link panda_link4: geometry collision mesh filename=package://franka_motion_control/assets/urdf/franka_descript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; visual mesh filename=package://franka_motion_control/assets/urdf/franka_descript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
- link panda_link5: geometry collision mesh filename=package://franka_motion_control/assets/urdf/franka_descript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; visual mesh filename=package://franka_motion_control/assets/urdf/franka_descript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
- link panda_link6: geometry collision mesh filename=package://franka_motion_control/assets/urdf/franka_descript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; visual mesh filename=package://franka_motion_control/assets/urdf/franka_descript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
- link panda_link7: geometry collision mesh filename=package://franka_motion_control/assets/urdf/franka_descript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; visual mesh filename=package://franka_motion_control/assets/urdf/franka_descript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
- link panda_rightfinger: geometry collision mesh filename=package://franka_motion_control/assets/urdf/franka_descript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; visual mesh filename=package://franka_motion_control/assets/urdf/franka_descript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

Commit message: fix link2 in urdf

File: assets/urdf/franka_description/franka_panda_no_gripper.urdf (robot description, URDF)
Before this commit: robot panda, 13 links, 12 joints
Links:
- removed link ee_link
- link panda_link2: geometry collision mesh filename=package://franka_motion_control/assets/urdf/franka_descript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; visual mesh filename=package://franka_motion_control/assets/urdf/franka_descript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
Joints:
- removed joint ee_fixed_joint
- joint panda_hand_joint: axis (none) -> 0 0 0; origin xyz=0 0 0.107 rpy=0 0 -0.785398163397 -> xyz=0 0 0.107 rpy=0 0 ${-pi/4}; parent panda_link7 -> panda_link8

Commit message: minor

File: assets/urdf/franka_description/franka_panda_no_gripper.urdf (robot description, URDF)
Before this commit: robot panda, 12 links, 11 joints
Joints:
- joint panda_hand_joint: parent panda_link8 -> panda_link7

Commit message: urdf cleanup

File: assets/urdf/franka_description/franka_panda_no_gripper.urdf (robot description, URDF)
Before this commit: robot panda, 12 links, 11 joints
Links:
- added link ee_link; collision box size=0.01 0.01 0.01
Joints:
- added joint ee_fixed_joint: type fixed, parent panda_hand, child ee_link, origin xyz=0.0 0. 0.1 rpy=0.0 0.0 ${-pi/2}
- joint panda_joint2: origin xyz=0 0 0 rpy=-1.57079632679 0 0 -> xyz=0 0 0 rpy=${-pi/2} 0 0
- joint panda_joint3: origin xyz=0 -0.316 0 rpy=1.57079632679 0 0 -> xyz=0 -0.316 0 rpy=${pi/2} 0 0
- joint panda_joint4: origin xyz=0.0825 0 0 rpy=1.57079632679 0 0 -> xyz=0.0825 0 0 rpy=${pi/2} 0 0
- joint panda_joint5: origin xyz=-0.0825 0.384 0 rpy=-1.57079632679 0 0 -> xyz=-0.0825 0.384 0 rpy=${-pi/2} 0 0
- joint panda_joint6: origin xyz=0 0 0 rpy=1.57079632679 0 0 -> xyz=0 0 0 rpy=${pi/2} 0 0
- joint panda_joint7: origin xyz=0.088 0 0 rpy=1.57079632679 0 0 -> xyz=0.088 0 0 rpy=${pi/2} 0 0

Commit message: make gripper open in urdf

File: assets/urdf/franka_description/franka_panda_no_gripper.urdf (robot description, URDF)
Before this commit: robot panda, 13 links, 12 joints
Joints:
- joint panda_finger_joint1: origin xyz=0 0 0.0584 rpy=0 0 0 -> xyz=0 0.04 0.0584 rpy=0 0 0
- joint panda_finger_joint2: origin xyz=0 0 0.0584 rpy=0 0 0 -> xyz=0 -0.04 0.0584 rpy=0 0 0
