Commit message: fixed franka urdf

File: assets/urdf/franka_description/deprecated/franka_panda_no_gripper.urdf (robot description, URDF)
Before this commit: robot panda, 14 links, 13 joints
Links:
- removed link panda_leftfinger
- removed link panda_link8
- removed link panda_rightfinger
- link panda_hand: geometry collision mesh filename=package://franka_motion_control/assets/urdf/franka_descript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; visual mesh filename=package://franka_motion_control/assets/urdf/franka_descript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
- link panda_link0: geometry collision mesh filename=package://franka_motion_control/assets/urdf/franka_descript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; visual mesh filename=package://franka_motion_control/assets/urdf/franka_descript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
- link panda_link1: geometry collision mesh filename=package://franka_motion_control/assets/urdf/franka_descript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; visual mesh filename=package://franka_motion_control/assets/urdf/franka_descript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
- link panda_link2: geometry collision mesh filename=package://franka_motion_control/assets/urdf/franka_descript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; visual mesh filename=package://franka_motion_control/assets/urdf/franka_descript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
- link panda_link3: geometry collision mesh filename=package://franka_motion_control/assets/urdf/franka_descript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; visual mesh filename=package://franka_motion_control/assets/urdf/franka_descript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
- link panda_link4: geometry collision mesh filename=package://franka_motion_control/assets/urdf/franka_descript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; visual mesh filename=package://franka_motion_control/assets/urdf/franka_descript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
- link panda_link5: geometry collision mesh filename=package://franka_motion_control/assets/urdf/franka_descript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; visual mesh filename=package://franka_motion_control/assets/urdf/franka_descript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
- link panda_link6: geometry collision mesh filename=package://franka_motion_control/assets/urdf/franka_descript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; visual mesh filename=package://franka_motion_control/assets/urdf/franka_descript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
- link panda_link7: geometry collision mesh filename=package://franka_motion_control/assets/urdf/franka_descript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; visual mesh filename=package://franka_motion_control/assets/urdf/franka_descript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
Joints:
- removed joint panda_finger_joint1
- removed joint panda_finger_joint2
- removed joint panda_joint8
- joint ee_fixed_joint: origin xyz=0.0 0. 0.1 rpy=0.0 0.0 -1.57 -> xyz=0.0 0. 0.1 rpy=0.0 0.0 ${-pi/2}
- joint panda_hand_joint: axis (none) -> 0 0 0; origin xyz=0 0 0 rpy=0 0 -0.785398163397 -> xyz=0 0 0.107 rpy=0 0 ${-pi/4}; parent panda_link8 -> panda_link7
- joint panda_joint2: origin xyz=0 0 0 rpy=-1.57079632679 0 0 -> xyz=0 0 0 rpy=${-pi/2} 0 0
- joint panda_joint3: origin xyz=0 -0.316 0 rpy=1.57079632679 0 0 -> xyz=0 -0.316 0 rpy=${pi/2} 0 0
- joint panda_joint4: origin xyz=0.0825 0 0 rpy=1.57079632679 0 0 -> xyz=0.0825 0 0 rpy=${pi/2} 0 0
- joint panda_joint5: origin xyz=-0.0825 0.384 0 rpy=-1.57079632679 0 0 -> xyz=-0.0825 0.384 0 rpy=${-pi/2} 0 0
- joint panda_joint6: origin xyz=0 0 0 rpy=1.57079632679 0 0 -> xyz=0 0 0 rpy=${pi/2} 0 0
- joint panda_joint7: origin xyz=0.088 0 0 rpy=1.57079632679 0 0 -> xyz=0.088 0 0 rpy=${pi/2} 0 0
